Commit message: Add scara_moveit_config and fix URDF mesh paths for MoveIt integration
- Fix package:// mesh references in scara_assembly.urdf (Scara Assembly1 -> scara_robot_pkg)
- Update STL meshes (Link_3, Link_4) from source
- Add scara_moveit_config package generated by MoveIt Setup Assistant
- Fix xacro macro name (spaces removed), add Joint_4 to arm group chain
- Add Joint_4 to all controller configs and initial_positions
- Add demo_with_controllers.launch.py for full ros2_control bringup

File: src/scara_robot_pkg/urdf/scara_assembly.urdf (robot description, URDF)
Before this commit: robot Scara Assembly urdf 1, 5 links, 4 joints
Links:
- link Link_3: mass 2.25445878305572 -> 2.2590769242565
- link Link_4: mass 0.004618141200777 -> 5.61232437594433E-05
Joints:
- joint Joint_2: origin xyz=0.65 0.0018761 0.275 rpy=0 0 0 -> xyz=0.65 0.00187609751792639 0.275 rpy=0 0 0
- joint Joint_3: origin xyz=0.6 0 0.88698 rpy=3.1416 0 0 -> xyz=0.6 0 0.886978614262261 rpy=3.14159265358979 0 0
