Commit message: Add dual-conveyor Gazebo pick-place pipeline

File: src/scara_robot_pkg/urdf/scara_gazebo.urdf.xacro (robot description, xacro)
@@ -38,5 +38,5 @@
         <parent link="world"/>
         <child link="base_link"/>
-        <origin xyz="0 -0.85 0" rpy="0 0 0"/>
+        <origin xyz="-1 0 0.8" rpy="0 0 0"/>
     </joint>
 </robot>
