Commit message: fix: absolute mesh paths, scene_publisher static objects, pick_place timeout

File: src/IFRA_ConveyorBelt/conveyorbelt_gazebo/urdf/chip.urdf (robot description, URDF)
Before this commit: robot chip, 1 links, 0 joints
Links:
- link base_link_chip: mass 0.0055 -> 4.40398679531101E-05; geometry collision mesh filename=file:///home/maxrec/projects/ros2-industrial-robot-simulati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; visual mesh filename=file:///home/maxrec/projects/ros2-industrial-robot-simulati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

File: src/IFRA_ConveyorBelt/conveyorbelt_gazebo/urdf/pcb.urdf (robot description, URDF)
Before this commit: robot pcb, 1 links, 0 joints
Links:
- removed link base_link_pcb
- added link base_link_PCB, mass 0.00030609; collision mesh filename=file:///home/maxrec/projects/ros2-industrial-robot-simulati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; visual mesh filename=file:///home/maxrec/projects/ros2-industrial-robot-simulati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
